File: projects/attenuator_10db/attenuator_10db.kicad_pcb (KiCad board)
At the start: 2 copper layers, 30 x 20 mm, 7 parts, among them J1 SMA_IN, J2 SMA_OUT

Commit message: feat: implement zoomed schematic render, CPWG controlled impedance synthesis, and custom circuit description parsing
Parts:
- R1, R3: value 96R -> 95.3R
- R2: value 71R -> 71.5R
- moved R2 2.80 mm to (15.0, 10.0)
- moved R1 0.91 mm to (10.5, 10.9), turned to -90 degrees
- moved R3 0.91 mm to (19.5, 10.9), turned to -90 degrees
Routing:
- net GND: track 0.00 -> 4.80 mm, vias 12 -> 28
- net RF_OUT: track 12.1 -> 9.59 mm
- net RF_IN: track 12.1 -> 9.59 mm
Other:
- board text added: "50Ω CPWG w=1.87 s=0.40"
- board text added: "PORT 1"
- board text added: "PORT 2"
- board text removed: "IN 50Ω"
- board text removed: "OUT 50Ω"
- board text removed: "Z0=50.0Ω"
